Commit message: URDF Rviz config
Arm task Rviz configuration

File: arm_urdf_new/arm_urdf_new/arm_urdf_new/urdf/Arm_urdf.urdf (robot description, URDF)
Before this commit: robot Arm_urdf, 11 links, 10 joints
Links:
- added link base_footprint; visual box size=0.001 0.001 0.001
- link arm_rotate: geometry collision mesh filename=package://arm_urdf_new/meshes/visual/arm_rotate.STL; visual mesh filename=package://arm_urdf_new/meshes/visual/arm_rotate.STL
- link base_link: geometry collision mesh filename=package://arm_urdf_new/meshes/visual/base_link.STL; visual mesh filename=package://arm_urdf_new/meshes/visual/base_link.STL
- link finger_1: geometry collision mesh filename=package://arm_urdf_new/meshes/visual/finger_1.STL; visual mesh filename=package://arm_urdf_new/meshes/visual/finger_1.STL
- link fingure_2: geometry collision mesh filename=package://arm_urdf_new/meshes/visual/fingure_2.STL; visual mesh filename=package://arm_urdf_new/meshes/visual/fingure_2.STL
- link lower_arm_cylinder: geometry collision mesh filename=package://arm_urdf_new/meshes/visual/lower_arm_cylinder.STL; visual mesh filename=package://arm_urdf_new/meshes/visual/lower_arm_cylinder.STL
- link red_block_1: geometry collision mesh filename=package://arm_urdf_new/meshes/visual/red_block_1.STL; visual mesh filename=package://arm_urdf_new/meshes/visual/red_block_1.STL
- link red_block_2: geometry collision mesh filename=package://arm_urdf_new/meshes/visual/red_block_2.STL; visual mesh filename=package://arm_urdf_new/meshes/visual/red_block_2.STL
- link shoulder_base: geometry collision mesh filename=package://arm_urdf_new/meshes/visual/shoulder_base.STL; visual mesh filename=package://arm_urdf_new/meshes/visual/shoulder_base.STL
- link supporter: geometry collision mesh filename=package://arm_urdf_new/meshes/visual/supporter.STL; visual mesh filename=package://arm_urdf_new/meshes/visual/supporter.STL
- link upper_arm_cylinder: geometry collision mesh filename=package://arm_urdf_new/meshes/visual/upper_arm_cylinder.STL; visual mesh filename=package://arm_urdf_new/meshes/visual/upper_arm_cylinder.STL
- link wrist_cylinder: geometry collision mesh filename=package://arm_urdf_new/meshes/visual/wrist_cylinder.STL; visual mesh filename=package://arm_urdf_new/meshes/visual/wrist_cylinder.STL
Joints:
- added joint base_footprint_joint: type fixed, parent base_footprint, child base_link, origin xyz=0 0 0.001 rpy=0 0 0
